Commit message: add caster for better stability

File: urdf/two_wheel_robot.urdf.xacro (robot description, xacro)
@@ -1,10 +1,12 @@
 <?xml version="1.0"?>
 <robot xmlns:xacro="http://www.ros.org/wiki/xacro" name="two_wheel_robot">
-  <xacro:property name="chassis_width" value="0.3"/>
-  <xacro:property name="chassis_length" value="0.4"/>
-  <xacro:property name="chassis_height" value="0.04"/>
-  <xacro:property name="wheel_radius" value="0.06"/>
+  <!-- 优化的参数配置 -->
+  <xacro:property name="chassis_width" value="0.35"/>    <!-- 增加宽度 -->
+  <xacro:property name="chassis_length" value="0.45"/>   <!-- 增加长度 -->
+  <xacro:property name="chassis_height" value="0.08"/>   <!-- 降低高度 -->
+  <xacro:property name="wheel_radius" value="0.12"/>
   <xacro:property name="wheel_width" value="0.05"/>
-  <xacro:property name="wheel_separation" value="0.35"/>
+  <xacro:property name="wheel_separation" value="0.30"/> <!-- 减小轮距 -->
+  <xacro:property name="caster_radius" value="0.025"/>   <!-- 脚轮半径 -->
   <!-- Base Link -->
   <link name="base_link"/>
@@ -21,5 +23,5 @@
     </visual>
     <collision>
-      <origin xyz="0 0 -0.03" rpy="0 0 0"/>
+      <origin xyz="0 0 0" rpy="0 0 0"/>
       <geometry>
         <box size="${chassis_length} ${chassis_width} ${chassis_height}"/>
@@ -27,6 +29,8 @@
     </collision>
     <inertial>
-      <mass value="15.0"/>
-      <inertia ixx="0.083" ixy="0.0" ixz="0.0" iyy="0.083" iyz="0.0" izz="0.083"/>
+      <mass value="12.0"/>  <!-- 增加质量 -->
+      <!-- 降低重心的惯性配置 -->
+      <origin xyz="0 0 -0.02" rpy="0 0 0"/>
+      <inertia ixx="0.15" ixy="0.0" ixz="0.0" iyy="0.25" iyz="0.0" izz="0.30"/>
     </inertial>
   </link>
@@ -34,5 +38,6 @@
     <parent link="base_link"/>
     <child link="chassis"/>
-    <origin xyz="0 0 ${wheel_radius}"/>
+    <!-- 调整底盘高度，使重心更低 -->
+    <origin xyz="0 0 ${wheel_radius + 0.01}"/>
   </joint>
   <!-- Left Wheel -->
@@ -54,6 +59,6 @@
     </collision>
     <inertial>
-      <mass value="1.0"/>
-      <inertia ixx="0.005" ixy="0.0" ixz="0.0" iyy="0.005" iyz="0.0" izz="0.01"/>
+      <mass value="1.5"/>  <!-- 增加轮子质量 -->
+      <inertia ixx="0.008" ixy="0.0" ixz="0.0" iyy="0.008" iyz="0.0" izz="0.015"/>
     </inertial>
   </link>
@@ -82,6 +87,6 @@
     </collision>
     <inertial>
-      <mass value="1.0"/>
-      <inertia ixx="0.005" ixy="0.0" ixz="0.0" iyy="0.005" iyz="0.0" izz="0.01"/>
+      <mass value="1.5"/>  <!-- 增加轮子质量 -->
+      <inertia ixx="0.008" ixy="0.0" ixz="0.0" iyy="0.008" iyz="0.0" izz="0.015"/>
     </inertial>
   </link>
@@ -92,4 +97,76 @@
     <axis xyz="0 1 0"/>
   </joint>
+  <!-- 前脚轮 -->
+  <link name="front_caster">
+    <visual>
+      <origin xyz="0 0 0" rpy="0 0 0"/>
+      <geometry>
+        <sphere radius="${caster_radius}"/>
+      </geometry>
+      <material name="grey">
+        <color rgba="0.5 0.5 0.5 1.0"/>
+      </material>
+    </visual>
+    <collision>
+      <origin xyz="0 0 0" rpy="0 0 0"/>
+      <geometry>
+        <sphere radius="${caster_radius}"/>
+      </geometry>
+      <!-- 降低摩擦力，让脚轮可以自由滑动 -->
+      <surface>
+        <friction>
+          <ode>
+            <mu>0.1</mu>
+            <mu2>0.1</mu2>
+          </ode>
+        </friction>
+      </surface>
+    </collision>
+    <inertial>
+      <mass value="0.2"/>
+      <inertia ixx="0.0001" ixy="0.0" ixz="0.0" iyy="0.0001" iyz="0.0" izz="0.0001"/>
+    </inertial>
+  </link>
+  <joint name="front_caster_joint" type="fixed">
+    <parent link="chassis"/>
+    <child link="front_caster"/>
+    <origin xyz="${chassis_length/2 - 0.08} 0 ${-chassis_height/2 - caster_radius - 0.005}" rpy="0 0 0"/>
+  </joint>
+  <!-- 后脚轮 -->
+  <link name="rear_caster">
+    <visual>
+      <origin xyz="0 0 0" rpy="0 0 0"/>
+      <geometry>
+        <sphere radius="${caster_radius}"/>
+      </geometry>
+      <material name="grey">
+        <color rgba="0.5 0.5 0.5 1.0"/>
+      </material>
+    </visual>
+    <collision>
+      <origin xyz="0 0 0" rpy="0 0 0"/>
+      <geometry>
+        <sphere radius="${caster_radius}"/>
+      </geometry>
+      <!-- 降低摩擦力，让脚轮可以自由滑动 -->
+      <surface>
+        <friction>
+          <ode>
+            <mu>0.1</mu>
+            <mu2>0.1</mu2>
+          </ode>
+        </friction>
+      </surface>
+    </collision>
+    <inertial>
+      <mass value="0.2"/>
+      <inertia ixx="0.0001" ixy="0.0" ixz="0.0" iyy="0.0001" iyz="0.0" izz="0.0001"/>
+    </inertial>
+  </link>
+  <joint name="rear_caster_joint" type="fixed">
+    <parent link="chassis"/>
+    <child link="rear_caster"/>
+    <origin xyz="${-chassis_length/2 + 0.08} 0 ${-chassis_height/2 - caster_radius - 0.005}" rpy="0 0 0"/>
+  </joint>
   <!-- Camera -->
   <link name="camera_link">
@@ -117,7 +194,8 @@
     <parent link="chassis"/>
     <child link="camera_link"/>
-    <origin xyz="${chassis_length/2} 0 ${chassis_height/2 + 0.05}" rpy="0 0 0"/>
-  </joint>
-  <!-- Gazebo Plugins -->
+    <!-- 降低相机高度，降低重心 -->
+    <origin xyz="${chassis_length/2} 0 ${chassis_height/2 + 0.025}" rpy="0 0 0"/>
+  </joint>
+  <!-- 优化的差分驱动控制器 -->
   <gazebo>
     <plugin name="differential_drive_controller" filename="libgazebo_ros_diff_drive.so">
@@ -125,49 +203,52 @@
         <namespace>/</namespace>
       </ros>
-      <update_rate>30</update_rate>
+      <update_rate>50</update_rate>  <!-- 提高更新频率 -->
       <left_joint>left_wheel_joint</left_joint>
       <right_joint>right_wheel_joint</right_joint>
       <wheel_separation>${wheel_separation}</wheel_separation>
       <wheel_diameter>${2*wheel_radius}</wheel_diameter>
-      <max_wheel_torque>20</max_wheel_torque>
-      <max_wheel_acceleration>1.0</max_wheel_acceleration>
+      <max_wheel_torque>35</max_wheel_torque>      <!-- 增加扭矩 -->
+      <max_wheel_acceleration>0.8</max_wheel_acceleration>  <!-- 降低加速度 -->
       <command_topic>cmd_vel</command_topic>
       <publish_odom>true</publish_odom>
       <publish_odom_tf>true</publish_odom_tf>
-      <publish_wheel_tf>false</publish_wheel_tf>
+      <publish_wheel_tf>true</publish_wheel_tf>
       <odometry_topic>odom</odometry_topic>
       <odometry_frame>odom</odometry_frame>
       <robot_base_frame>base_link</robot_base_frame>
+      <!-- 添加噪声模型，更真实的仿真 -->
+      <wheel_torque>35</wheel_torque>
+      <wheel_acceleration>0.8</wheel_acceleration>
     </plugin>
   </gazebo>
   <!-- Camera Plugin -->
   <gazebo reference="camera_link">
-    <sensor type="camera" name="camera">           <!-- 1. 传感器定义 -->
-      <update_rate>30.0</update_rate>              <!-- 2. 更新频率 -->
-      <camera name="head">                         <!-- 3. 相机参数组 -->
-        <horizontal_fov>1.3962634</horizontal_fov> <!-- 4. 视场角 -->
-        <image>                                    <!-- 5. 图像参数 -->
-          <width>640</width>                       <!-- 图像宽度 -->
-          <height>480</height>                     <!-- 图像高度 -->
-          <format>R8G8B8</format>                  <!-- 像素格式 -->
+    <sensor type="camera" name="camera">
+      <update_rate>30.0</update_rate>
+      <camera name="head">
+        <horizontal_fov>1.3962634</horizontal_fov>
+        <image>
+          <width>640</width>
+          <height>480</height>
+          <format>R8G8B8</format>
         </image>
-        <clip>                                     <!-- 6. 裁剪距离 -->
-          <near>0.02</near>                        <!-- 最近距离 -->
-          <far>300</far>                           <!-- 最远距离 -->
+        <clip>
+          <near>0.02</near>
+          <far>300</far>
         </clip>
       </camera>
-      <plugin name="camera_controller" filename="libgazebo_ros_camera.so"> <!-- 7. ROS2插件 -->
+      <plugin name="camera_controller" filename="libgazebo_ros_camera.so">
         <ros>
           <namespace>/</namespace>
-          <remapping>image_raw:=robot_camera/image_raw</remapping>        <!-- 8. 话题重映射 -->
+          <remapping>image_raw:=robot_camera/image_raw</remapping>
           <remapping>camera_info:=robot_camera/camera_info</remapping>
         </ros>
-        <camera_name>robot_camera</camera_name>    <!-- 9. 相机名称 -->
-        <frame_name>camera_link</frame_name>       <!-- 10. TF坐标系 -->
-        <hack_baseline>0.07</hack_baseline>        <!-- 11. 立体视觉参数 -->
+        <camera_name>robot_camera</camera_name>
+        <frame_name>camera_link</frame_name>
+        <hack_baseline>0.07</hack_baseline>
       </plugin>
     </sensor>
   </gazebo>
-  <!-- Colors for Gazebo -->
+  <!-- Gazebo材质 -->
   <gazebo reference="chassis">
     <material>Gazebo/Blue</material>
@@ -175,7 +256,25 @@
   <gazebo reference="left_wheel">
     <material>Gazebo/DarkGrey</material>
+    <!-- 增加轮子摩擦力 -->
+    <mu1>1.0</mu1>
+    <mu2>1.0</mu2>
   </gazebo>
   <gazebo reference="right_wheel">
     <material>Gazebo/DarkGrey</material>
+    <!-- 增加轮子摩擦力 -->
+    <mu1>1.0</mu1>
+    <mu2>1.0</mu2>
+  </gazebo>
+  <gazebo reference="front_caster">
+    <material>Gazebo/Grey</material>
+    <!-- 脚轮低摩擦 -->
+    <mu1>0.1</mu1>
+    <mu2>0.1</mu2>
+  </gazebo>
+  <gazebo reference="rear_caster">
+    <material>Gazebo/Grey</material>
+    <!-- 脚轮低摩擦 -->
+    <mu1>0.1</mu1>
+    <mu2>0.1</mu2>
   </gazebo>
   <gazebo reference="camera_link">

Commit message: further change caster to show in gazebo

File: urdf/two_wheel_robot.urdf.xacro (robot description, xacro)
@@ -267,14 +267,22 @@
   </gazebo>
   <gazebo reference="front_caster">
-    <material>Gazebo/Grey</material>
+    <material>Gazebo/White</material>
     <!-- 脚轮低摩擦 -->
-    <mu1>0.1</mu1>
-    <mu2>0.1</mu2>
+    <mu1>0.05</mu1>
+    <mu2>0.05</mu2>
+    <kp>1000000.0</kp>
+    <kd>100.0</kd>
+    <minDepth>0.001</minDepth>
+    <maxVel>1.0</maxVel>
   </gazebo>
   <gazebo reference="rear_caster">
-    <material>Gazebo/Grey</material>
+    <material>Gazebo/White</material>
     <!-- 脚轮低摩擦 -->
-    <mu1>0.1</mu1>
-    <mu2>0.1</mu2>
+    <mu1>0.05</mu1>
+    <mu2>0.05</mu2>
+    <kp>1000000.0</kp>
+    <kd>100.0</kd>
+    <minDepth>0.001</minDepth>
+    <maxVel>1.0</maxVel>
   </gazebo>
   <gazebo reference="camera_link">

Commit message: further change of caster and chassis

File: urdf/two_wheel_robot.urdf.xacro (robot description, xacro)
@@ -4,9 +4,9 @@
   <xacro:property name="chassis_width" value="0.35"/>    <!-- 增加宽度 -->
   <xacro:property name="chassis_length" value="0.45"/>   <!-- 增加长度 -->
-  <xacro:property name="chassis_height" value="0.08"/>   <!-- 降低高度 -->
+  <xacro:property name="chassis_height" value="0.06"/>   <!-- 降低高度 -->
   <xacro:property name="wheel_radius" value="0.12"/>
   <xacro:property name="wheel_width" value="0.05"/>
-  <xacro:property name="wheel_separation" value="0.30"/> <!-- 减小轮距 -->
-  <xacro:property name="caster_radius" value="0.025"/>   <!-- 脚轮半径 -->
+  <xacro:property name="wheel_separation" value="0.35"/> <!-- 减小轮距 -->
+  <xacro:property name="caster_radius" value="0.08"/>   <!-- 脚轮半径 -->
   <!-- Base Link -->
   <link name="base_link"/>
@@ -124,5 +124,5 @@
     </collision>
     <inertial>
-      <mass value="0.2"/>
+      <mass value="0.8"/>
       <inertia ixx="0.0001" ixy="0.0" ixz="0.0" iyy="0.0001" iyz="0.0" izz="0.0001"/>
     </inertial>
@@ -160,5 +160,5 @@
     </collision>
     <inertial>
-      <mass value="0.2"/>
+      <mass value="0.8"/>
       <inertia ixx="0.0001" ixy="0.0" ixz="0.0" iyy="0.0001" iyz="0.0" izz="0.0001"/>
     </inertial>

Commit message: decreaase caster radius as it was too large~!

File: urdf/two_wheel_robot.urdf.xacro (robot description, xacro)
@@ -8,5 +8,5 @@
   <xacro:property name="wheel_width" value="0.05"/>
   <xacro:property name="wheel_separation" value="0.35"/> <!-- 减小轮距 -->
-  <xacro:property name="caster_radius" value="0.08"/>   <!-- 脚轮半径 -->
+  <xacro:property name="caster_radius" value="0.06"/>   <!-- 脚轮半径 -->
   <!-- Base Link -->
   <link name="base_link"/>
